File: HARDWARE/MCU_And_IMU.kicad_sch (KiCad schematic)
At the start: 16 parts, among them SW1 SW_SPST, U2 STM32G431KBTx, Y1 Crystal_GND24

Commit message: Add other fields to BOM
Parts:
- C10, C11: DigiKey Part # (none) -> 311-1014-1-ND; MANUFACTURER (none) -> YAGEO; MFN CC0402JRNPO9BN100 -> (none); Mfg Part # (none) -> CC0402JRNPO9BN100; Package (none) -> 0402; Part Number 311-1014-1-ND -> (none)
- C12, C5, C6, C7, C8, C9: DigiKey Part # (none) -> 1276-6720-1-ND; MANUFACTURER (none) -> Samsung Electro-Mechanics; MFN CL05B104KA5NNNC -> (none); Mfg Part # (none) -> CL05B104KA5NNNC; Package (none) -> 0402; Part Number 1276-6720-1-ND -> (none)
- LED1: DigiKey Part # (none) -> 754-1506-1-ND; MANUFACTURER (none) -> Kingbright; MFN APHBM2012QBDSURKC -> (none); Mfg Part # (none) -> APHBM2012QBDSURKC; Package (none) -> 0805; Part Number 754-1506-1-ND -> (none)
- MT1: DigiKey Part # (none) -> 1428-1152-1-ND; MFN ICM-42605 -> (none); Mfg Part # (none) -> ICM-42605; Package (none) -> 14-LGA; Part Number 1428-1152-1-ND -> (none)
- R3, R5: DigiKey Part # (none) -> 311-10KJRCT-ND; MANUFACTURER (none) -> YAGEO; MFN RC0402JR-0710KL -> (none); Mfg Part # (none) -> RC0402JR-0710KL; Package (none) -> 0402; Part Number 311-10KJRCT-ND -> (none)
- R4: DigiKey Part # (none) -> 311-68.0LRCT-ND; MANUFACTURER (none) -> YAGEO; MFN RC0402FR-0768RL -> (none); Mfg Part # (none) -> RC0402FR-0768RL; Package (none) -> 0402; Part Number 311-68.0LRCT-ND -> (none)
- SW1: DigiKey Part # (none) -> 2508-R-667995TR-ND; MANUFACTURER (none) -> Mitsumi Electric Company Ltd; MFN R-667995 -> (none); Mfg Part # (none) -> R-667995; Package (none) -> SMT; Part Number 2508-R-667995TR-ND -> (none)
- U2: DigiKey Part # (none) -> 497-19470-ND; MANUFACTURER (none) -> STMicroelectronics; MFN STM32G431KBT6 -> (none); Mfg Part # (none) -> STM32G431KBT6; Package (none) -> 32-QFP; Part Number 497-19470-ND -> (none)
- Y1: DigiKey Part # (none) -> 50-ECS-160-10-36-CKM-TR3TR-ND; MANUFACTURER (none) -> ECS Inc.; MFN ECS-160-10-36-CKM-TR3 -> (none); Mfg Part # (none) -> ECS-160-10-36-CKM-TR3; Package (none) -> 4-SMD; Part Number 50-ECS-160-10-36-CKM-TR3TR-ND -> (none)

Commit message: Clean up routing and layout
Other:
- note added: "Crystal C_{L} = 10pF Assume C_{stray} ~= 5pF C_{10} = C_{11} = 2*(C_{L}-C_{stray}) = 10pF From app note AN2867"
- note added: "nRST pin controlled by SWD interface Add C12 for debounce and R3 for a stronger pull-up Both these components are optional"
- note removed: "Crystal C_{L} = 10pF Assume C_{stray} ~= 5pF C_{L1} = C_{L2} = 2*(C_{L}-C_{stray}) = 10pF From app note AN2867"
- note removed: "nRST pin controlled by SWD interface Add C11 for debounce and R3 for a stronger pull-up Both these components are optional"
Changed lines of the file:
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@@
 		)
 	)
-	(text "nRST pin controlled by SWD interface\nAdd C11 for debounce and R3 for a stronger pull-up\nBoth these components are optional"
+	(text "nRST pin controlled by SWD interface\nAdd C12 for debounce and R3 for a stronger pull-up\nBoth these components are optional"
 		(exclude_from_sim no)
 		(at 35.56 151.638 0)
@@
 		)
 	)
-	(text "Crystal C_{L} = 10pF\nAssume C_{stray} ~= 5pF\nC_{L1} = C_{L2} = 2*(C_{L}-C_{stray}) = 10pF\nFrom app note AN2867"
+	(text "Crystal C_{L} = 10pF\nAssume C_{stray} ~= 5pF\nC_{10} = C_{11} = 2*(C_{L}-C_{stray}) = 10pF\nFrom app note AN2867"
 		(exclude_from_sim no)
 		(at 38.354 65.024 0)
